Commit message: buller_core

File: catkin_ws/src/buller_description/urdf/buller.urdf (robot description, URDF)
Before this commit: robot buller, 3 links, 2 joints
Links:
- link base_link: geometry visual cylinder length=0.562 radius=0.15
Joints:
- joint base_to_left_wheel: origin xyz=-0.09 -0.2005 -0.235 -> xyz=-0.09 -0.10 -0.281
- joint base_to_right_wheel: origin xyz=-0.09 0.2005 -0.235 -> xyz=-0.09 0.10 -0.281
